Commit message: adapted urdf and moveit configuration to biomaz project

File: z1_description/urdf/z1.urdf.xacro (robot description, xacro)
@@ -5,5 +5,6 @@
     <xacro:arg name="controllers" default="$(find z1_bringup)/config/z1_controllers.yaml" />
     <xacro:arg name="sim_ignition" default="true" />
-    <xacro:arg name="with_gripper" default="true" />
+    <!-- kept only for compatibility, no longer used -->
+    <xacro:arg name="with_gripper" default="false" />
     <xacro:include filename="$(find z1_description)/urdf/const.xacro" />
     <xacro:include filename="$(find z1_description)/urdf/z1.ros2_control.xacro" />
@@ -27,6 +28,5 @@
         <collision>
             <geometry>
-                <mesh filename="package://z1_description/meshes/collision/z1_Link00.STL"
-                    scale="1 1 1" />
+                <mesh filename="package://z1_description/meshes/collision/z1_Link00.STL" scale="1 1 1" />
             </geometry>
             <origin rpy="0 0 0" xyz="0 0 ${motor_height/2.0}" />
@@ -47,6 +47,5 @@
         <axis xyz="0 0 1" />
         <dynamics damping="${jointDamping}" friction="${jointFriction}" />
-        <limit effort="${torqueMax}" velocity="${velocityMax}" lower="${joint1_PositionMin}"
-            upper="${joint1_PositionMax}" />
+        <limit effort="${torqueMax}" velocity="${velocityMax}" lower="${joint1_PositionMin}" upper="${joint1_PositionMax}" />
     </joint>
     <link name="link01">
@@ -60,6 +59,5 @@
         <collision>
             <geometry>
-                <mesh filename="package://z1_description/meshes/collision/z1_Link01.STL"
-                    scale="1 1 1" />
+                <mesh filename="package://z1_description/meshes/collision/z1_Link01.STL" scale="1 1 1" />
             </geometry>
         </collision>
@@ -79,6 +77,5 @@
         <axis xyz="0 1 0" />
         <dynamics damping="${2*jointDamping}" friction="${2*jointFriction}" />
-        <limit effort="${2*torqueMax}" velocity="${velocityMax}" lower="${joint2_PositionMin}"
-            upper="${joint2_PositionMax}" />
+        <limit effort="${2*torqueMax}" velocity="${velocityMax}" lower="${joint2_PositionMin}" upper="${joint2_PositionMax}" />
     </joint>
     <link name="link02">
@@ -92,6 +89,5 @@
         <collision>
             <geometry>
-                <mesh filename="package://z1_description/meshes/collision/z1_Link02.STL"
-                    scale="1 1 1" />
+                <mesh filename="package://z1_description/meshes/collision/z1_Link02.STL" scale="1 1 1" />
             </geometry>
         </collision>
@@ -111,6 +107,5 @@
         <axis xyz="0 1 0" />
         <dynamics damping="${jointDamping}" friction="${jointFriction}" />
-        <limit effort="${torqueMax}" velocity="${velocityMax}" lower="${joint3_PositionMin}"
-            upper="${joint3_PositionMax}" />
+        <limit effort="${torqueMax}" velocity="${velocityMax}" lower="${joint3_PositionMin}" upper="${joint3_PositionMax}" />
     </joint>
     <link name="link03">
@@ -124,6 +119,5 @@
         <collision>
             <geometry>
-                <mesh filename="package://z1_description/meshes/collision/z1_Link03.STL"
-                    scale="1 1 1" />
+                <mesh filename="package://z1_description/meshes/collision/z1_Link03.STL" scale="1 1 1" />
             </geometry>
         </collision>
@@ -143,6 +137,5 @@
         <axis xyz="0 1 0" />
         <dynamics damping="${jointDamping}" friction="${jointFriction}" />
-        <limit effort="${torqueMax}" velocity="${velocityMax}" lower="${joint4_PositionMin}"
-            upper="${joint4_PositionMax}" />
+        <limit effort="${torqueMax}" velocity="${velocityMax}" lower="${joint4_PositionMin}" upper="${joint4_PositionMax}" />
     </joint>
     <link name="link04">
@@ -156,6 +149,5 @@
         <collision>
             <geometry>
-                <mesh filename="package://z1_description/meshes/collision/z1_Link04.STL"
-                    scale="1 1 1" />
+                <mesh filename="package://z1_description/meshes/collision/z1_Link04.STL" scale="1 1 1" />
             </geometry>
         </collision>
@@ -175,6 +167,5 @@
         <axis xyz="0 0 1" />
         <dynamics damping="${jointDamping}" friction="${jointFriction}" />
-        <limit effort="${torqueMax}" velocity="${velocityMax}" lower="${joint5_PositionMin}"
-            upper="${joint5_PositionMax}" />
+        <limit effort="${torqueMax}" velocity="${velocityMax}" lower="${joint5_PositionMin}" upper="${joint5_PositionMax}" />
     </joint>
     <link name="link05">
@@ -188,6 +179,5 @@
         <collision>
             <geometry>
-                <mesh filename="package://z1_description/meshes/collision/z1_Link05.STL"
-                    scale="1 1 1" />
+                <mesh filename="package://z1_description/meshes/collision/z1_Link05.STL" scale="1 1 1" />
             </geometry>
         </collision>
@@ -207,6 +197,5 @@
         <axis xyz="1 0 0" />
         <dynamics damping="${jointDamping}" friction="${jointFriction}" />
-        <limit effort="${torqueMax}" velocity="${velocityMax}" lower="${joint6_PositionMin}"
-            upper="${joint6_PositionMax}" />
+        <limit effort="${torqueMax}" velocity="${velocityMax}" lower="${joint6_PositionMin}" upper="${joint6_PositionMax}" />
     </joint>
     <link name="link06">
@@ -220,6 +209,5 @@
         <collision>
             <geometry>
-                <mesh filename="package://z1_description/meshes/collision/z1_Link06.STL"
-                    scale="1 1 1" />
+                <mesh filename="package://z1_description/meshes/collision/z1_Link06.STL" scale="1 1 1" />
             </geometry>
         </collision>
@@ -233,74 +221,36 @@
         </inertial>
     </link>
-    <xacro:if value="$(arg with_gripper)">
-        <joint name="gripperStatorLink" type="fixed">
-            <origin rpy="0 0 0" xyz="0.051 0.0 0.0" />
-            <parent link="link06" />
-            <child link="gripperStator" />
-        </joint>
-        <link name="gripperStator">
-            <visual>
-                <geometry>
-                    <mesh filename="package://z1_description/meshes/visual/z1_GripperStator.dae"
-                        scale="1 1 1" />
-                </geometry>
-                <material name="Grey" />
-            </visual>
-            <collision>
-                <geometry>
-                    <mesh filename="package://z1_description/meshes/collision/z1_GripperStator.STL"
-                        scale="1 1 1" />
-                </geometry>
-            </collision>
-            <inertial>
-                <origin rpy="0 0 0"
-                    xyz="${GripperStator_ComX} ${GripperStator_ComY} ${GripperStator_ComZ}" />
-                <mass value="${GripperStator_Mass}" />
-                <inertia
-                    ixx="${GripperStator_Ixx}" ixy="${GripperStator_Ixy}" ixz="${GripperStator_Ixz}"
-                    iyy="${GripperStator_Iyy}" iyz="${GripperStator_Iyz}"
-                    izz="${GripperStator_Izz}" />
-            </inertial>
-        </link>
-        <joint name="jointGripper" type="revolute">
-            <origin rpy="0 0 0" xyz="0.049 0.0 0" />
-            <parent link="gripperStator" />
-            <child link="gripperMover" />
-            <axis xyz="0 1 0" />
-            <dynamics damping="${jointDamping}" friction="${jointFriction}" />
-            <limit effort="${torqueMax}" velocity="${velocityMax}" lower="${Gripper_PositionMin}"
-                upper="${Gripper_PositionMax}" />
-        </joint>
-        <link name="gripperMover">
-            <visual>
-                <geometry>
-                    <mesh filename="package://z1_description/meshes/visual/z1_GripperMover.dae"
-                        scale="1 1 1" />
-                </geometry>
-                <material name="Grey" />
-            </visual>
-            <collision>
-                <geometry>
-                    <mesh filename="package://z1_description/meshes/collision/z1_GripperMover.STL"
-                        scale="1 1 1" />
-                </geometry>
-            </collision>
-            <inertial>
-                <origin rpy="0 0 0"
-                    xyz="${GripperMover_ComX} ${GripperMover_ComY} ${GripperMover_ComZ}" />
-                <mass value="${GripperMover_Mass}" />
-                <inertia
-                    ixx="${GripperMover_Ixx}" ixy="${GripperMover_Ixy}" ixz="${GripperMover_Ixz}"
-                    iyy="${GripperMover_Iyy}" iyz="${GripperMover_Iyz}"
-                    izz="${GripperMover_Izz}" />
-            </inertial>
-        </link>
-        <gazebo reference="gripperStator">
-            <self_collide>true</self_collide>
-        </gazebo>
-        <gazebo reference="gripperMover">
-            <self_collide>true</self_collide>
-        </gazebo>
-    </xacro:if>
+    <!-- Pollinator tool -->
+    <joint name="jointPollinatorTool" type="fixed">
+        <origin rpy="0 0 0" xyz="0.18 0.0 0.0" />
+        <parent link="link06" />
+        <child link="pollinatorTool" />
+    </joint>
+    <link name="pollinatorTool">
+        <visual>
+            <origin rpy="0 1.57079632679 0" xyz="-0.07 0 0" />
+            <geometry>
+                <cylinder radius="0.0075" length="0.14" />
+            </geometry>
+            <material name="Grey" />
+        </visual>
+        <collision>
+            <origin rpy="0 1.57079632679 0" xyz="-0.07 0 0" />
+            <geometry>
+                <cylinder radius="0.0075" length="0.14" />
+            </geometry>
+        </collision>
+        <inertial>
+            <origin rpy="0 0 0" xyz="-0.07 0 0" />
+            <mass value="0.10" />
+            <inertia
+                ixx="0.000165"
+                ixy="0.0"
+                ixz="0.0"
+                iyy="0.000165"
+                iyz="0.0"
+                izz="0.000003" />
+        </inertial>
+    </link>
     <xacro:if value="$(arg sim_ignition)">
         <gazebo reference="world" />
@@ -319,4 +269,4 @@
         prefix="$(arg prefix)"
         sim_ignition="$(arg sim_ignition)"
-        with_gripper="$(arg with_gripper)" />
+        with_gripper="false" />
 </robot>

Commit message: added D405 camera

File: z1_description/urdf/z1.urdf.xacro (robot description, xacro)
@@ -9,4 +9,5 @@
     <xacro:include filename="$(find z1_description)/urdf/const.xacro" />
     <xacro:include filename="$(find z1_description)/urdf/z1.ros2_control.xacro" />
+    <xacro:include filename="$(find realsense2_description)/urdf/_d405.urdf.xacro" />
     <material name="Grey">
         <color rgba="0.3 0.3 0.3 1.0" />
@@ -253,4 +254,7 @@
         </inertial>
     </link>
+    <xacro:sensor_d405 parent="link06" use_nominal_extrinsics="true">
+        <origin xyz="0.12 0 -0.02" rpy="0 0 0"/>
+    </xacro:sensor_d405>
     <xacro:if value="$(arg sim_ignition)">
         <gazebo reference="world" />
