Commit message: modified robot world frame

File: z1_description/urdf/z1.urdf.xacro (robot description, xacro)
@@ -13,8 +13,8 @@
         <color rgba="0.3 0.3 0.3 1.0" />
     </material>
-    <link name="world" />
+    <link name="arm_base" />
     <joint name="base_static_joint" type="fixed">
         <origin rpy="0 0 0" xyz="0 0 0" />
-        <parent link="world" />
+        <parent link="arm_base" />
         <child link="link00" />
     </joint>
@@ -258,5 +258,5 @@
     </xacro:sensor_d405>
     <xacro:if value="$(arg sim_ignition)">
-        <gazebo reference="world" />
+        <gazebo reference="arm_base" />
         <gazebo>
             <plugin filename="libign_ros2_control-system.so"
