Commit message: modified joint 2 limits

File: z1_description/urdf/const.xacro (robot description, xacro)
@@ -109,5 +109,5 @@
     <xacro:property name="joint1_PositionMin" value="${-PI*150/180}"/>
     <xacro:property name="joint1_PositionMax" value="${PI*150/180}"/>
-    <xacro:property name="joint2_PositionMin" value="0.0"/>
+    <xacro:property name="joint2_PositionMin" value="-0.01"/>
     <xacro:property name="joint2_PositionMax" value="${PI*170/180}"/>
     <xacro:property name="joint3_PositionMin" value="${-PI*165/180}"/>
